File: hardware/board.sch (EAGLE design)
At the start: 25 parts, among them IC1 NCP1117ST33T3G, SW1 SWITCH-2P, SW2 SWITCH-2P, SW3 SWITCH

Commit message: feat: .gitignore file for hardware directory
Parts:
- removed D1: RGB-5050, WorTel2023:RGB-5050
- removed POWER: SOCKET-C, WorTel2023:SOCKET-C
- removed R10, R8, R9: 100, Resistor:R_CHIP-0805(2012-METRIC)
- removed R7: 470, Resistor:R_CHIP-0805(2012-METRIC)
- removed SW3: SWITCH, XLKM#4:SWITCH
- removed UART: PINHD-1X04_1X04M, Tinkercad:PINHD-1X04_1X04M
- added C4: 1µ, Capacitor:C_CHIP-0805(2012-METRIC)
- added C5: 100n, Capacitor:C_CHIP-0805(2012-METRIC)
- added J1: CSP-USC16-TR, CSP-USC16-TR:CSP-USC16-TR
- added NEO1: WS2812B, LED:WS2812B
- added Q1, Q2: BSS138, Transistor:NMOSFETSOT23-GSD
- added U1: CH340C, CH340C:CH340C
- R5, R6: value 470 -> 5.1K
Connections:
- removed net +5V_FUSE: F1.2, POWER.V-BUS
- removed net N$3: D1.5, R8.2
- removed net N$7: R7.1, SW3.1
- removed net RXD: ESP-12E/F.RXD, UART.3
- removed net TXD: ESP-12E/F.TXD, UART.2
- new net +5V_BF: BREAKOUT.1, F1.2, J1.VBUS_A, J1.VBUS_B
- new net ESP_RX: BREAKOUT.5, ESP-12E/F.RXD
- new net ESP_TX: BREAKOUT.4, ESP-12E/F.TXD, U1.RXD
- new net EXP_RX: U1.TXD
- new net N$1: J1.DP1, J1.DP2, U1.UD+
- new net N$8: Q1.G, Q2.S, U1.!RTS
- net +3.3V: now also BREAKOUT.2, C5.1, U1.V3, U1.VCC; no longer BREAKOUT.3, SW3.2
- net +5V: now also NEO1.VDD; no longer BREAKOUT.2, UART.4
- net GND: now also BREAKOUT.3, C4.2, C5.2, J1.SHELL_GND, NEO1.VSS, R5.1, R6.1, U1.GND; no longer BREAKOUT.1, D1.1, D1.2, D1.3, POWER.GND, POWER.SHIELD, UART.1
- net IO0: now also Q1.D, SW1.1; no longer R5.1
- net IO12: now also BREAKOUT.11; no longer BREAKOUT.10, R10.1
- net IO13: now also BREAKOUT.9; no longer BREAKOUT.8, R8.1
- net IO14: now also BREAKOUT.10, NEO1.DIN; no longer BREAKOUT.9, R9.1
- net IO15: no longer BREAKOUT.4, R7.2
- net IO16: no longer BREAKOUT.11
- net IO2: now also BREAKOUT.6; no longer BREAKOUT.5
- net IO4: now also BREAKOUT.7; no longer BREAKOUT.6
- net IO5: now also BREAKOUT.8; no longer BREAKOUT.7
- net N$2: now also J1.DN1, J1.DN2, U1.UD-; no longer D1.4, R10.2
- net N$4: now also Q1.S, Q2.G, U1.!DTR; no longer D1.6, R9.2
- net N$5: now also J1.CC2; no longer SW1.1
- net N$6: now also J1.CC1; no longer SW2.1
- net RST: now also C4.1, Q2.D, SW2.1; no longer R6.1
Other:
- moved on the sheet: F1, R5, R6
